File: vca_main_board/mcu.sch (KiCad schematic (older format))
At the start: 3 parts, among them U4 STM32H743VITx

Commit message: done
Parts:
- removed IC?: STM32G474QET6, Package_QFP:LQFP-128_14x14mm_P0.4mm, symbol STM32G474QET6:STM32G474QET6
- removed U4: STM32H743VITx, Package_QFP:LQFP-100_14x14mm_P0.5mm, symbol MCU_ST_STM32H7:STM32H743VITx
- added C20, C24, C25, C26, C27, C28, C29, C52: 100n 6.3V, Capacitor_SMD:C_0603_1608Metric_Pad1.08x0.95mm_HandSolder, symbol Device:C_Small
- added C21, C22: 2u2 6.3V, Capacitor_SMD:C_0603_1608Metric_Pad1.08x0.95mm_HandSolder, symbol Device:C_Small
- added C30: 1u 6.3V, Capacitor_SMD:C_0603_1608Metric_Pad1.08x0.95mm_HandSolder, symbol Device:C_Small
- added C41, C58: 4.7u 6.3V, Capacitor_SMD:C_0603_1608Metric_Pad1.08x0.95mm_HandSolder, symbol Device:C_Small
- added D10: ESDA6V1BC6, Package_TO_SOT_SMD:SOT-23-6_Handsoldering, symbol Power_Protection:ESDA6V1BC6
- added J3: SWD, 10pin_1.27_socket:10pin_1.27_socket, symbol Connector:Conn_ARM_JTAG_SWD_10
- added R4: 47k 5%, Resistor_SMD:R_0603_1608Metric_Pad0.98x0.95mm_HandSolder, symbol Device:R_Small
- added R41: 1k 5%, Resistor_SMD:R_0603_1608Metric_Pad0.98x0.95mm_HandSolder, symbol Device:R_Small
- added SW1: RST, Button_Switch_THT:SW_PUSH_6mm_H4.3mm, symbol Switch:SW_Push
- added U6: STM32H743VITx, Package_QFP:LQFP-100_14x14mm_P0.5mm, symbol MCU_ST_STM32H7:STM32H743VITx
- added Y1: 10MHz, Crystal:Resonator_SMD_muRata_CSTxExxV-3Pin_3.0x1.1mm_HandSoldering, symbol Device:Crystal_GND2_Small
- C23: renamed from C?; value 1u/10V -> 100n 6.3V
Connections:
- net +3V3: now reaches C23.1
- net +3V3: now also C24.1, C25.1, C26.1, C27.1, C28.1, C29.1, C30.1, C41.1, C52.1, C58.1, J3.1 (VTref), U6.100 (VDD), U6.11 (VDD), U6.21 (VDDA), U6.27 (VDD), U6.50 (VDD), U6.6 (VBAT), U6.75 (VDD)
- net GND: now reaches C23.2
- net GND: now also C20.2, C21.2, C22.2, C24.2, C25.2, C26.2, C27.2, C28.2, C29.2, C30.2, C41.2, C52.2, C58.2, D10.2 (COM), D10.5 (COM), J3.3 (GND), J3.5 (GND), J3.9 (GNDDetect), R4.1, R41.2, U6.10 (VSS), U6.19 (VSSA), U6.26 (VSS), U6.49 (VSS), U6.74 (VSS), U6.99 (VSS), Y1.2
- new net: U6.12 (PH0), Y1.1
- new net: U6.13 (PH1), Y1.3
- new net: C21.1, U6.48 (VCAP1)
- new net: C22.1, U6.73 (VCAP2)
- new net: R41.1, SW1.1
- new net BOOT0: R4.2, U6.94 (BOOT0)
- new net BUZZ: U6.45 (PE15)
- new net CAN_FAULT: U6.96 (PB9)
- new net CAN_S: U6.95 (PB8)
- new net COIL_FANS: U6.68 (PA9)
- new net COIL_TH_1: U6.31 (PA7)
- new net COIL_TH_2: U6.33 (PC5)
- new net EEP_~WC: U6.9 (PC15)
- new net EXTA_0: U6.81 (PD0)
- new net EXTA_1: U6.82 (PD1)
- new net EXTA_2: U6.83 (PD2)
- new net EXTA_3: U6.86 (PD5)
- new net EXTA_4: U6.87 (PD6)
- new net EXTA_5: U6.67 (PA8)
- new net EXTA_6: U6.66 (PC9)
- new net EXTA_7: U6.25 (PA3)
- new net EXTB_0: U6.97 (PE0)
- new net EXTB_1: U6.98 (PE1)
- new net EXTB_2: U6.1 (PE2)
- new net EXTB_3: U6.2 (PE3)
- new net EXTB_4: U6.3 (PE4)
- new net EXTB_5: U6.4 (PE5)
- new net EXTB_6: U6.5 (PE6)
- new net EXTB_7: U6.37 (PE7)
- new net EXTRA_FAN_1: U6.40 (PE10)
- new net EXTRA_FAN_2: U6.41 (PE11)
- new net EXT_GPIO_A: U6.91 (PB5)
- new net EXT_GPIO_B: U6.65 (PC8)
- new net FDCAN_RX: U6.51 (PB12)
- new net FDCAN_TX: U6.52 (PB13)
- new net H_CURR: U6.18 (PC3_C)
- new net H_Excitation: U6.28 (PA4)
- new net H_Load_H: U6.30 (PA6)
- new net H_Offset: U6.29 (PA5)
- new net H_REF_HIGH: U6.24 (PA2)
- new net H_Sum: U6.32 (PC4)
- new net H_Th: U6.35 (PB1)
- new net H_VOLT: U6.22 (PA0)
- new net Knob_A: U6.59 (PD12)
- new net Knob_B: U6.60 (PD13)
- new net Knob_S: U6.34 (PB0)
- new net LCD_BL: U6.8 (PC14)
- new net LCD_CLK: U6.46 (PB10)
- new net LCD_CS: U6.90 (PB4)
- new net LCD_DC: U6.80 (PC12)
- new net LCD_DIN: U6.16 (PC1)
- new net LCD_RST: U6.7 (PC13)
- new net LED_1: U6.53 (PB14)
- new net LED_2: U6.54 (PB15)
- new net MIRROR_ENC_A: U6.77 (PA15)
- new net MIRROR_ENC_B: U6.23 (PA1)
- new net MIRROR_ENC_Z: U6.63 (PC6)
- new net NRST: C20.1, D10.3 (TVS2), J3.10 (~RESET~), SW1.2, U6.14 (NRST)
- new net SCL: U6.92 (PB6)
- new net SDA: U6.93 (PB7)
- new net SWDCLK: D10.6 (TVS4), J3.4 (SWDCLK/TCK), U6.76 (PA14)
- new net SWDIO: D10.4 (TVS3), J3.2 (SWDIO/TMS), U6.72 (PA13)
- new net SWO: D10.1 (TVS1), J3.6 (SWO/TDO), U6.89 (PB3)
- new net TH_ALERT: U6.47 (PB11)
- new net USB_DET: U6.69 (PA10)
- new net USB_RX: U6.71 (PA12)
- new net USB_TX: U6.70 (PA11)
- new net VREF: U6.20 (VREF+)
- no-connect marks 0 -> 21
Other:
- note added: "MCU"
- note added: "STM32H743VIT6"
- note added: "SWD"
- moved on the sheet: C23
