File: vca_main_board/power.sch (KiCad schematic (older format))
At the start: 36 parts, among them J1 KPJX-4S-S, J2 Power terminal, Q1 STB15N80K5, Q2 STB15N80K5, SW1 POW_SWITCH, U1 173010335, U2 173010535, U3 173011235

Commit message: done
Parts:
- removed C1, C10, C2, C3, C4, C5, C6: 4u7/50V, Capacitor_SMD:C_1210_3225Metric_Pad1.33x2.70mm_HandSolder, symbol Device:C_Small
- removed C14, C17: 22u/25V, Capacitor_SMD:C_1210_3225Metric_Pad1.33x2.70mm_HandSolder, symbol Device:C_Small
- removed J1: KPJX-4S-S, KPJX-4S-S:KPJX-4S-S, symbol KPJX-4S-S:KPJX-4S-S
- removed JP1: Jumper_NC, Jumper:SolderJumper-2_P1.3mm_Bridged_Pad1.0x1.5mm, symbol Device:Jumper_NC_Small
- removed L3: XAL4030-472, Inductor_SMD:L_Coilcraft_XxL4030, symbol Device:L_Small
- removed Q1, Q2: STB15N80K5, Package_TO_SOT_SMD:TO-263-2, symbol Transistor_FET:STB15N80K5
- removed SW1: POW_SWITCH, Connector_Wire:SolderWire-0.5sqmm_1x02_P4.6mm_D0.9mm_OD2.1mm_Relief, symbol Switch:SW_SPST
- removed U3: 173011235, 17301xx35:17301xx35, symbol 17301xx35:17301xx35
- added C5, C6: 180u 50V, Capacitor_SMD:CP_Elec_8x10.5, symbol Device:CP_Small
- added D2: 10A 60V, Package_TO_SOT_SMD:TO-252-2, symbol Device:D_Schottky_AKA
- added J1: 12V_OUT, TerminalBlock_Phoenix:TerminalBlock_Phoenix_PT-1,5-2-5.0-H_1x02_P5.00mm_Horizontal, symbol Connector:Screw_Terminal_01x02
- added Q1: IRF740, Package_TO_SOT_THT:TO-220-3_Horizontal_TabDown, symbol Transistor_FET:IRF740
- added TP1, TP2, TP3, TP4: GND, TestPoint:TestPoint_Loop_D2.60mm_Drill1.6mm_Beaded, symbol Connector:TestPoint
- C11, C12, C7, C8, C9: value 4u7/50V -> 10u 20V; footprint Capacitor_SMD:C_1210_3225Metric_Pad1.33x2.70mm_HandSolder -> Capacitor_SMD:C_1206_3216Metric_Pad1.33x1.80mm_HandSolder
- C13, C15, C16, C18: value 22u/25V -> 22u 10V
- D1: value LED -> LED GREEN
- F1: value Fuse 4A -> Fuse 500mA
- F2: value Fuse 4A -> Fuse 1A
- J2: value Power terminal -> 12V_IN
- R1: value 100k 1% -> 47k 5%
- R2: value 100k 1% -> 100k 5%
Connections:
- net +VDC is gone; now on net +12V: L1.1, L2.1, R3.1
- net +12V: now also C7.1, C8.1, C9.1, F1.1, F2.1, R2.1, C5.1, C6.1; no longer C15.1, C18.1
- net +5V: now also C15.1, C18.1
- net GND: now also R1.2, C5.2, C6.2, D2.1 (A), D2.3 (A), J1.2 (Pin_2), Q1.3 (S), TP1.1, TP2.1, TP3.1, TP4.1
- net at L1.2, U1.1 (VIN): now also C11.1; no longer C7.1
- net at F1.2: now also J1.1 (Pin_1)
- net at J2.1 (Pin_1): now also F2.2
- net at J2.2 (Pin_2): now also Q1.2 (D); no longer F2.2
- net at R2.2: now also R1.1, D2.2 (K), Q1.1 (G)
- net at L2.2, U2.1 (VIN): now also C12.1; no longer C11.1, C8.1
Other:
- note added: "Additional power output"
- note added: "GND test points"
- note added: "Integrated buck converters (1A out)"
- note added: "Main power input"
- note added: "Power indicator LED"
- note added: "Primary rail capacitors"
- note removed: "+VDC rail is 20V DC sourced from GSM120A20-R7B"
- note removed: "Main power connector"
- note removed: "Mean Well GSM120A20-R7B \npower supply side"
- moved on the sheet: C13, C16, D1, F2, J2, L1, R2, R3, U1, U2
